Commit message: Add rpilidar dependency; update URDF to include scan frame

File: jrb_description/urdf/robotrouge.urdf (robot description, URDF)
Before this commit: robot robotrouge, 21 links, 20 joints
Links:
- added link laser_link
Joints:
- added joint laser_join: type fixed, parent base_link, child laser_link, origin xyz=0.0 0.0 0.37733 rpy=0 0 0

File: jrb_description/urdf/robotrouge.urdf.xacro (robot description, xacro)
@@ -57,4 +57,10 @@
     </visual>
   </link>
+  <joint name="laser_join" type="fixed">
+    <parent link="base_link" />
+    <child link="laser_link" />
+    <origin xyz="0.0 0.0 0.37733" rpy="0 0 0"/>
+  </joint>
+  <link name="laser_link" />
   <joint name="wheel_left_joint" type="continuous">
     <parent link="base_link"/>

Commit message: Rename jrb_sample_detector to jrb_sensors; add obstacle_detector

File: jrb_description/urdf/robotrouge.urdf (robot description, URDF)
Before this commit: robot robotrouge, 22 links, 21 joints
Joints:
- removed joint laser_join
- added joint laser_joint: type fixed, parent base_link, child laser_link, origin xyz=0.0 0.0 0.37733 rpy=0 0 -1.5707963267948966

File: jrb_description/urdf/robotrouge.urdf.xacro (robot description, xacro)
@@ -57,8 +57,8 @@
     </visual>
   </link>
-  <joint name="laser_join" type="fixed">
+  <joint name="laser_joint" type="fixed">
     <parent link="base_link" />
     <child link="laser_link" />
-    <origin xyz="0.0 0.0 0.37733" rpy="0 0 0"/>
+    <origin xyz="0.0 0.0 0.37733" rpy="0 0 ${radians(-90)}"/>
   </joint>
   <link name="laser_link" />
