Commit message: wip actuators

File: jrb_description/urdf/arm.urdf.xacro (robot description, xacro)
@@ -28,5 +28,5 @@
       <origin xyz="${xyz}" rpy="0 0 0" />
       <axis xyz="0 0 1" />
-      <limit effort="30" velocity="1.0" lower="-0.056" upper="0.056" />
+      <limit effort="30" velocity="1.0" lower="0.0" upper="0.224" />
     </joint>
     <link
@@ -45,8 +45,8 @@
     <joint
       name="${name}_b_joint"
-      type="continuous">
+      type="revolute">
       <origin
         xyz="0.02814995 0 0"
-        rpy="0 0 0" />
+        rpy="0 0 ${radians(135)}" />
       <parent
         link="${name}_arm_base_link" />
@@ -55,4 +55,5 @@
       <axis
         xyz="0 0 1" />
+      <limit effort="30" velocity="1.0" lower="${radians(135)}" upper="${radians(315)}" />
     </joint>
     <link name="${name}_c">
@@ -67,9 +68,10 @@
       </visual>
     </link>
-    <joint name="${name}_c_joint" type="continuous">
+    <joint name="${name}_c_joint" type="revolute">
       <origin xyz="0.054 0 0" rpy="0 0 0" />
       <parent link="${name}_b" />
       <child link="${name}_c" />
-      <axis xyz="0 0 -1" />
+      <axis xyz="0 0 1" />
+      <limit effort="30" velocity="1.0" lower="${radians(-90)}" upper="${radians(90)}" />
     </joint>
     <link name="${name}_d">
@@ -82,9 +84,10 @@
       </visual>
     </link>
-    <joint name="${name}_d_joint" type="continuous">
+    <joint name="${name}_d_joint" type="revolute">
       <origin xyz="0.031 0 -0.009" rpy="0 0 0" />
       <parent link="${name}_c" />
       <child link="${name}_d" />
       <axis xyz="0 1 0" />
+      <limit effort="30" velocity="1.0" lower="0" upper="${radians(-90)}" />
     </joint>
     <link
@@ -100,8 +103,8 @@
     <joint
       name="${name}_e_joint"
-      type="continuous">
+      type="revolute">
       <origin
         xyz="0.0319 0 0"
-        rpy="0 0 0" />
+        rpy="${radians(-90)} 0 0" />
       <parent
         link="${name}_d" />
@@ -109,5 +112,6 @@
         link="${name}_e" />
       <axis
-        xyz="0  0 1" />
+        xyz="1 0 0" />
+      <limit effort="30" velocity="1.0" lower="${radians(-90)}" upper="${radians(90)}" />
     </joint>
     <link

File: jrb_description/urdf/robotrouge.urdf (robot description, URDF)
Before this commit: robot robotrouge, 19 links, 18 joints
Joints:
- joint base_joint: origin xyz=0.0 0.0 0.01416 rpy=0 0 0 -> xyz=0.0 0.0 0.0147 rpy=0 0 0
- joint left_arm_joint: limit lower=-0.056 upper=0.056 effort=30 velocity=1.0 -> lower=0.0 upper=0.224 effort=30 velocity=1.0; origin xyz=0.054 0.11275 0.141375 rpy=0 0 0 -> xyz=0.054 0.11275 0.029375 rpy=0 0 0
- joint left_b_joint: limit (none) -> lower=2.356194490192345 upper=5.497787143782138 effort=30 velocity=1.0; origin xyz=0.02814995 0 0 rpy=0 0 0 -> xyz=0.02814995 0 0 rpy=0 0 2.356194490192345; type continuous -> revolute
- joint left_c_joint: axis 0 0 -1 -> 0 0 1; limit (none) -> lower=-1.5707963267948966 upper=1.5707963267948966 effort=30 velocity=1.0; type continuous -> revolute
- joint left_d_joint: limit (none) -> lower=0 upper=-1.5707963267948966 effort=30 velocity=1.0; type continuous -> revolute
- joint left_e_joint: axis 0  0 1 -> 1 0 0; limit (none) -> lower=-1.5707963267948966 upper=1.5707963267948966 effort=30 velocity=1.0; origin xyz=0.0319 0 0 rpy=0 0 0 -> xyz=0.0319 0 0 rpy=-1.5707963267948966 0 0; type continuous -> revolute
- joint right_arm_joint: limit lower=-0.056 upper=0.056 effort=30 velocity=1.0 -> lower=0.0 upper=0.224 effort=30 velocity=1.0; origin xyz=0.054 -0.11275 0.141375 rpy=0 0 0 -> xyz=0.054 -0.11275 0.029375 rpy=0 0 0
- joint right_b_joint: limit (none) -> lower=2.356194490192345 upper=5.497787143782138 effort=30 velocity=1.0; origin xyz=0.02814995 0 0 rpy=0 0 0 -> xyz=0.02814995 0 0 rpy=0 0 2.356194490192345; type continuous -> revolute
- joint right_c_joint: axis 0 0 -1 -> 0 0 1; limit (none) -> lower=-1.5707963267948966 upper=1.5707963267948966 effort=30 velocity=1.0; type continuous -> revolute
- joint right_d_joint: limit (none) -> lower=0 upper=-1.5707963267948966 effort=30 velocity=1.0; type continuous -> revolute
- joint right_e_joint: axis 0  0 1 -> 1 0 0; limit (none) -> lower=-1.5707963267948966 upper=1.5707963267948966 effort=30 velocity=1.0; origin xyz=0.0319 0 0 rpy=0 0 0 -> xyz=0.0319 0 0 rpy=-1.5707963267948966 0 0; type continuous -> revolute
- joint th_camera_joint: origin xyz=0.091 0.0 0.3183 rpy=0 0 0 -> xyz=0.1468 0.0 0.317 rpy=0 0 0
- joint wheel_left_joint: origin xyz=0.0 0.08316 0 rpy=-1.57 0 0 -> xyz=0.0 0.08316 0.01004 rpy=-1.57 0 0
- joint wheel_right_joint: origin xyz=0.0 -0.08316  0.0 rpy=-1.57 0 0 -> xyz=0.0 -0.08316  0.01004 rpy=-1.57 0 0

File: jrb_description/urdf/robotrouge.urdf.xacro (robot description, xacro)
@@ -137,5 +137,5 @@
   </link>
   <!-- Arms -->
-  <xacro:arm name="left" xyz="0.054 0.11275 0.141375"/>
-  <xacro:arm name="right" xyz="0.054 -0.11275 0.141375"/>
+  <xacro:arm name="left" xyz="0.054 0.11275 0.029375"/>
+  <xacro:arm name="right" xyz="0.054 -0.11275 0.029375"/>
 </robot>

Commit message: arm_to_sample ok !

File: jrb_description/urdf/arm.urdf.xacro (robot description, xacro)
@@ -7,5 +7,11 @@
     <color rgba="0.792156862745098 0.819607843137255 0.933333333333333 1" />
   </material>
-  <xacro:macro name="arm" params="name xyz">
+  <xacro:macro name="arm" params="name xyz origin">
+    <link name="${name}_arm_origin_link" />
+    <joint name="${name}_arm_origin_joint" type="fixed">
+      <parent link="base_link"/>
+      <child link="${name}_arm_origin_link"/>
+      <origin xyz="${origin}" rpy="0 0 ${radians(-90)}"/>
+    </joint>
     <link
       name="${name}_arm_base_link">
@@ -47,6 +53,5 @@
       type="revolute">
       <origin
-        xyz="0.02814995 0 0"
-        rpy="0 0 ${radians(135)}" />
+        xyz="0.02814995 0 0" rpy="0 0 ${radians(150)}" />
       <parent
         link="${name}_arm_base_link" />
@@ -54,6 +59,6 @@
         link="${name}_b" />
       <axis
-        xyz="0 0 1" />
-      <limit effort="30" velocity="1.0" lower="${radians(135)}" upper="${radians(315)}" />
+        xyz="0 0 -1" />
+      <limit effort="30" velocity="1.0" lower="${radians(0)}" upper="${radians(300)}" />
     </joint>
     <link name="${name}_c">
@@ -69,9 +74,9 @@
     </link>
     <joint name="${name}_c_joint" type="revolute">
-      <origin xyz="0.054 0 0" rpy="0 0 0" />
+      <origin xyz="0.054 0 0" rpy="0 0 ${radians(-150)}" />
       <parent link="${name}_b" />
       <child link="${name}_c" />
       <axis xyz="0 0 1" />
-      <limit effort="30" velocity="1.0" lower="${radians(-90)}" upper="${radians(90)}" />
+      <limit effort="30" velocity="1.0" lower="${radians(0)}" upper="${radians(300)}" />
     </joint>
     <link name="${name}_d">
@@ -85,9 +90,9 @@
     </link>
     <joint name="${name}_d_joint" type="revolute">
-      <origin xyz="0.031 0 -0.009" rpy="0 0 0" />
+      <origin xyz="0.031 0 -0.009" rpy="0 ${radians(-150+90)} 0" />
       <parent link="${name}_c" />
       <child link="${name}_d" />
       <axis xyz="0 1 0" />
-      <limit effort="30" velocity="1.0" lower="0" upper="${radians(-90)}" />
+      <limit effort="30" velocity="1.0" lower="${radians(0)}" upper="${radians(300)}" />
     </joint>
     <link
@@ -105,6 +110,5 @@
       type="revolute">
       <origin
-        xyz="0.0319 0 0"
-        rpy="${radians(-90)} 0 0" />
+        xyz="0.0319 0 0" rpy="${radians(-240)} 0 0" />
       <parent
         link="${name}_d" />
@@ -113,5 +117,5 @@
       <axis
         xyz="1 0 0" />
-      <limit effort="30" velocity="1.0" lower="${radians(-90)}" upper="${radians(90)}" />
+      <limit effort="30" velocity="1.0" lower="${radians(0)}" upper="${radians(300)}" />
     </joint>
     <link

File: jrb_description/urdf/robotrouge.urdf (robot description, URDF)
Before this commit: robot robotrouge, 19 links, 18 joints
Links:
- added link left_arm_origin_link
- added link right_arm_origin_link
Joints:
- added joint left_arm_origin_joint: type fixed, parent base_link, child left_arm_origin_link, origin xyz=0.0865 0.11275 0 rpy=0 0 -1.5707963267948966
- added joint right_arm_origin_joint: type fixed, parent base_link, child right_arm_origin_link, origin xyz=0.0865 -0.11275 0 rpy=0 0 -1.5707963267948966
- joint left_b_joint: axis 0 0 1 -> 0 0 -1; limit lower=2.356194490192345 upper=5.497787143782138 effort=30 velocity=1.0 -> lower=0.0 upper=5.235987755982989 effort=30 velocity=1.0; origin xyz=0.02814995 0 0 rpy=0 0 2.356194490192345 -> xyz=0.02814995 0 0 rpy=0 0 2.6179938779914944
- joint left_c_joint: limit lower=-1.5707963267948966 upper=1.5707963267948966 effort=30 velocity=1.0 -> lower=0.0 upper=5.235987755982989 effort=30 velocity=1.0; origin xyz=0.054 0 0 rpy=0 0 0 -> xyz=0.054 0 0 rpy=0 0 -2.6179938779914944
- joint left_d_joint: limit lower=0 upper=-1.5707963267948966 effort=30 velocity=1.0 -> lower=0.0 upper=5.235987755982989 effort=30 velocity=1.0; origin xyz=0.031 0 -0.009 rpy=0 0 0 -> xyz=0.031 0 -0.009 rpy=0 -1.0471975511965976 0
- joint left_e_joint: limit lower=-1.5707963267948966 upper=1.5707963267948966 effort=30 velocity=1.0 -> lower=0.0 upper=5.235987755982989 effort=30 velocity=1.0; origin xyz=0.0319 0 0 rpy=-1.5707963267948966 0 0 -> xyz=0.0319 0 0 rpy=-4.1887902047863905 0 0
- joint right_b_joint: axis 0 0 1 -> 0 0 -1; limit lower=2.356194490192345 upper=5.497787143782138 effort=30 velocity=1.0 -> lower=0.0 upper=5.235987755982989 effort=30 velocity=1.0; origin xyz=0.02814995 0 0 rpy=0 0 2.356194490192345 -> xyz=0.02814995 0 0 rpy=0 0 2.6179938779914944
- joint right_c_joint: limit lower=-1.5707963267948966 upper=1.5707963267948966 effort=30 velocity=1.0 -> lower=0.0 upper=5.235987755982989 effort=30 velocity=1.0; origin xyz=0.054 0 0 rpy=0 0 0 -> xyz=0.054 0 0 rpy=0 0 -2.6179938779914944
- joint right_d_joint: limit lower=0 upper=-1.5707963267948966 effort=30 velocity=1.0 -> lower=0.0 upper=5.235987755982989 effort=30 velocity=1.0; origin xyz=0.031 0 -0.009 rpy=0 0 0 -> xyz=0.031 0 -0.009 rpy=0 -1.0471975511965976 0
- joint right_e_joint: limit lower=-1.5707963267948966 upper=1.5707963267948966 effort=30 velocity=1.0 -> lower=0.0 upper=5.235987755982989 effort=30 velocity=1.0; origin xyz=0.0319 0 0 rpy=-1.5707963267948966 0 0 -> xyz=0.0319 0 0 rpy=-4.1887902047863905 0 0

File: jrb_description/urdf/robotrouge.urdf.xacro (robot description, xacro)
@@ -137,5 +137,5 @@
   </link>
   <!-- Arms -->
-  <xacro:arm name="left" xyz="0.054 0.11275 0.029375"/>
-  <xacro:arm name="right" xyz="0.054 -0.11275 0.029375"/>
+  <xacro:arm name="left" xyz="0.054 0.11275 0.029375" origin="0.0865 0.11275 0"/>
+  <xacro:arm name="right" xyz="0.054 -0.11275 0.029375" origin="0.0865 -0.11275 0"/>
 </robot>
