Commit message: wip

File: jrb_description/urdf/arm.urdf.xacro (robot description, xacro)
@@ -1,3 +1,3 @@
-<?xml version="1.0" ?>
+<?xml version="1.0"?>
 <robot xmlns:xacro="http://ros.org/wiki/xacro">
   <material name="arm_yellow">
@@ -10,7 +10,7 @@
     <link name="${name}_arm_origin_link" />
     <joint name="${name}_arm_origin_joint" type="fixed">
-      <parent link="base_link"/>
-      <child link="${name}_arm_origin_link"/>
-      <origin xyz="${origin}" rpy="0 0 ${radians(-90)}"/>
+      <parent link="base_link" />
+      <child link="${name}_arm_origin_link" />
+      <origin xyz="${origin}" rpy="0 0 ${radians(-90)}" />
     </joint>
     <link
@@ -22,5 +22,5 @@
         <geometry>
           <mesh
-            filename="package://jrb_description/meshes/${name}_arm_base_link.STL" />
+            filename="package://jrb_description/urdf/meshes/${name}_arm_base_link.STL" />
         </geometry>
         <material name="arm_black">
@@ -44,5 +44,5 @@
         <geometry>
           <mesh
-            filename="package://jrb_description/meshes/${name}_bras.STL" />
+            filename="package://jrb_description/urdf/meshes/${name}_bras.STL" />
         </geometry>
         <material name="arm_yellow" />
@@ -68,5 +68,5 @@
           rpy="0 0 0" />
         <geometry>
-          <mesh filename="package://jrb_description/meshes/${name}_avant_bras.STL" />
+          <mesh filename="package://jrb_description/urdf/meshes/${name}_avant_bras.STL" />
         </geometry>
         <material name="arm_gray" />
@@ -84,5 +84,5 @@
         <origin xyz="0 0 0" rpy="0 0 0" />
         <geometry>
-          <mesh filename="package://jrb_description/meshes/poignet.STL" />
+          <mesh filename="package://jrb_description/urdf/meshes/poignet.STL" />
         </geometry>
         <material name="arm_gray" />
@@ -101,5 +101,5 @@
         <origin xyz="0 0 0" rpy="0 0 0" />
         <geometry>
-          <mesh filename="package://jrb_description/meshes/${name}_prehenseur.STL" />
+          <mesh filename="package://jrb_description/urdf/meshes/${name}_prehenseur.STL" />
         </geometry>
         <material name="arm_yellow" />
@@ -127,5 +127,5 @@
         <geometry>
           <mesh
-            filename="package://jrb_description/meshes/ventouse.STL" />
+            filename="package://jrb_description/urdf/meshes/ventouse.STL" />
         </geometry>
         <material name="arm_gray" />

File: jrb_description/urdf/robotrouge.urdf.xacro (robot description, xacro)
@@ -1,147 +1,371 @@
-<?xml version="1.0" ?>
+<?xml version="1.0"?>
 <robot name="robotrouge"
   xmlns:xacro="http://ros.org/wiki/xacro">
-  <xacro:include filename="arm.urdf.xacro" />
-  <!-- Init colour -->
-  <material name="black">
-      <color rgba="0.0 0.0 0.0 1.0"/>
-  </material>
-  <material name="dark">
-    <color rgba="0.3 0.3 0.3 1.0"/>
-  </material>
-  <material name="light_black">
-    <color rgba="0.4 0.4 0.4 1.0"/>
-  </material>
-  <material name="blue">
-    <color rgba="0.0 0.0 0.8 1.0"/>
-  </material>
-  <material name="green">
-    <color rgba="0.0 0.8 0.0 1.0"/>
-  </material>
-  <material name="grey">
-    <color rgba="0.5 0.5 0.5 1.0"/>
-  </material>
-  <material name="orange">
-    <color rgba="1.0 0.4235 0.0392 1.0"/>
-  </material>
-  <material name="brown">
-    <color rgba="0.8706 0.8118 0.7647 1.0"/>
-  </material>
-  <material name="red">
-    <color rgba="0.8 0.0 0.0 1.0"/>
-  </material>
-  <material name="white">
-    <color rgba="1.0 1.0 1.0 1.0"/>
-  </material>
-  <link name="base_footprint"/>
+  <!-- <xacro:include filename="arm.urdf.xacro" /> -->
+  <xacro:include filename="colors.xacro" />
+  <xacro:include filename="inertial.xacro" />
+  <!-- Webots -->
+  <webots>
+    <device reference="laser_link" type="Lidar">
+      <ros>
+        <enabled>true</enabled>
+        <updateRate>5</updateRate>
+        <topicName>/scan</topicName>
+        <alwaysOn>true</alwaysOn>
+        <frameName>laser_link</frameName>
+      </ros>
+    </device>
+    <plugin type="webots_ros2_control::Ros2Control" />
+  </webots>
+  <ros2_control name="WebotsControl" type="system">
+    <hardware>
+      <plugin>webots_ros2_control::Ros2ControlSystem</plugin>
+    </hardware>
+    <joint name="right_wheel_joint">
+      <state_interface name="position" />
+      <command_interface name="velocity" />
+    </joint>
+    <joint name="left_wheel_joint">
+      <state_interface name="position" />
+      <command_interface name="velocity" />
+    </joint>
+  </ros2_control>
+  <!-- BASE LINK -->
+  <link name="chassis">
+    <visual>
+      <origin xyz="0 0 0.075" />
+      <geometry>
+        <box size="0.3 0.3 0.15" />
+      </geometry>
+      <material name="white" />
+    </visual>
+    <collision>
+      <origin xyz="0 0 0.075" />
+      <geometry>
+        <box size="0.3 0.3 0.15" />
+      </geometry>
+    </collision>
+    <xacro:inertial_box mass="0.5" x="0.3" y="0.3" z="0.15">
+      <origin xyz="0 0 0.075" rpy="0 0 0" />
+    </xacro:inertial_box>
+  </link>
+  <!-- LEFT WHEEL LINK -->
+  <joint name="left_wheel_joint" type="continuous">
+    <parent link="chassis" />
+    <child link="left_wheel" />
+    <origin xyz="0 0.15 0" rpy="-${pi/2} 0 0" />
+    <axis xyz="0 0 1" />
+  </joint>
+  <link name="left_wheel">
+    <visual>
+      <geometry>
+        <cylinder radius="0.0254" length="0.02" />
+      </geometry>
+      <material name="blue" />
+    </visual>
+    <collision>
+      <geometry>
+        <cylinder radius="0.0254" length="0.02" />
+      </geometry>
+    </collision>
+    <xacro:inertial_cylinder mass="0.1" length="0.02" radius="0.0254">
+      <origin xyz="0 0 0" rpy="0 0 0" />
+    </xacro:inertial_cylinder>
+  </link>
+  <!-- RIGHT WHEEL LINK -->
+  <joint name="right_wheel_joint" type="continuous">
+    <parent link="chassis" />
+    <child link="right_wheel" />
+    <origin xyz="0 -0.15 0" rpy="${pi/2} 0 0" />
+    <axis xyz="0 0 -1" />
+  </joint>
+  <link name="right_wheel">
+    <visual>
+      <geometry>
+        <cylinder radius="0.0254" length="0.02" />
+      </geometry>
+      <material name="blue" />
+    </visual>
+    <collision>
+      <geometry>
+        <cylinder radius="0.0254" length="0.02" />
+      </geometry>
+    </collision>
+    <xacro:inertial_cylinder mass="0.1" length="0.02" radius="0.0254">
+      <origin xyz="0 0 0" rpy="0 0 0" />
+    </xacro:inertial_cylinder>
+  </link>
+  <!-- FRONT CASTER WHEEL LINK -->
+  <joint name="front_caster_wheel_joint" type="fixed">
+    <parent link="chassis" />
+    <child link="front_caster_wheel" />
+    <origin xyz="0.12 0 0" />
+  </joint>
+  <link name="front_caster_wheel">
+    <visual>
+      <geometry>
+        <sphere radius="0.0254" />
+      </geometry>
+      <material name="black" />
+    </visual>
+    <collision>
+      <geometry>
+        <sphere radius="0.0254" />
+      </geometry>
+    </collision>
+    <xacro:inertial_sphere mass="0.1" radius="0.0254">
+      <origin xyz="0 0 0" rpy="0 0 0" />
+    </xacro:inertial_sphere>
+  </link>
+  <!-- BACK CASTER WHEEL LINK -->
+  <joint name="back_caster_wheel_joint" type="fixed">
+    <parent link="chassis" />
+    <child link="back_caster_wheel" />
+    <origin xyz="-0.12 0 0" />
+  </joint>
+  <link name="back_caster_wheel">
+    <visual>
+      <geometry>
+        <sphere radius="0.0254" />
+      </geometry>
+      <material name="black" />
+    </visual>
+    <collision>
+      <geometry>
+        <sphere radius="0.0254" />
+      </geometry>
+    </collision>
+    <xacro:inertial_sphere mass="0.1" radius="0.0254">
+      <origin xyz="0 0 0" rpy="0 0 0" />
+    </xacro:inertial_sphere>
+  </link>
+  <!-- LASER LINK  -->
+  <joint name="laser_joint" type="fixed">
+    <parent link="chassis" />
+    <child link="laser_link" />
+    <origin xyz="0.0 0.0 0.37733" rpy="0 0 ${-pi/2}" />
+  </joint>
+  <link name="laser_link">
+    <visual>
+      <origin xyz="0 0 0" rpy="0 0 0" />
+      <geometry>
+        <box size="0.02 0.02 0.001" />
+      </geometry>
+      <material name="dark" />
+    </visual>
+    <collision>
+      <origin xyz="0 0 0" rpy="0 0 0" />
+      <geometry>
+        <box size="0.02 0.02 0.001" />
+      </geometry>
+      <material name="dark" />
+    </collision>
+  </link>
+  <!-- <link name="base_footprint">
+    <visual>
+      <origin xyz="0 0 0.02" rpy="0 0 0" />
+      <geometry>
+        <mesh filename="package://jrb_description/urdf/meshes/carter.STL" />
+      </geometry>
+    </visual>
+    <collision>
+      <origin xyz="0 0 0.22" rpy="0 0 0" />
+      <geometry>
+        <box size="0.2 0.27 0.4" />
+      </geometry>
+      <material name="light_black" />
+    </collision>
+  </link>
   <joint name="base_joint" type="fixed">
-    <parent link="base_footprint"/>
-    <child link="base_link"/>
-    <origin xyz="0.0 0.0 0.0147" rpy="0 0 0"/>
+    <parent link="base_footprint" />
+    <child link="base_link" />
+    <origin xyz="0.0 0.0 0.0147" rpy="0 0 0" />
   </joint>
   <link name="base_link">
     <visual>
-      <!-- <origin xyz="-0.032 0 0.0147" rpy="0 0 0"/> -->
-      <origin xyz="0 0 -0.003" rpy="0 0 3.14"/>
-      <geometry>
-        <!-- <box size="0.140 0.140 0.143"/> -->
-        <mesh filename="package://jrb_description/meshes/base.STL" />
-      </geometry>
-      <material name="light_black"/>
-    </visual>
-    <visual>
-      <origin xyz="0 0 0" rpy="0 0 0"/>
-      <geometry>
-        <mesh filename="package://jrb_description/meshes/carter.STL" />
-      </geometry>
-    </visual>
+      <origin xyz="0 0 -0.003" rpy="0 0 3.14" />
+      <geometry>
+        <mesh filename="package://jrb_description/urdf/meshes/base.STL" />
+      </geometry>
+      <material name="light_black" />
+    </visual>
+    <collision>
+      <origin xyz="0 0 0" rpy="0 0 0" />
+      <geometry>
+        <box size="0.2 0.27 0.01" />
+      </geometry>
+      <material name="light_black" />
+    </collision>
+  </link>
+  <joint name="caster_front_joint" type="fixed">
+    <parent link="base_footprint" />
+    <child link="caster_front_link" />
+    <origin rpy="0 0 0" xyz="0.09 0.0 0.01" />
+  </joint>
+  <link name="caster_front_link">
+    <visual>
+      <origin rpy="0 0 0" xyz="0 0 0" />
+      <geometry>
+        <sphere radius="0.01" />
+      </geometry>
+      <material name="Black" />
+    </visual>
+    <collision>
+      <geometry>
+        <sphere radius="0.01" />
+      </geometry>
+      <origin rpy="0 0 0" xyz="0 0 0" />
+    </collision>
+  </link>
+  <joint name="caster_back_joint" type="fixed">
+    <parent link="base_footprint" />
+    <child link="caster_back_link" />
+    <origin rpy="0 0 0" xyz="-0.09 0.0 0.01" />
+  </joint>
+  <link name="caster_back_link">
+    <visual>
+      <origin rpy="0 0 0" xyz="0 0 0" />
+      <geometry>
+        <sphere radius="0.01" />
+      </geometry>
+      <material name="Black" />
+    </visual>
+    <collision>
+      <geometry>
+        <sphere radius="0.01" />
+      </geometry>
+      <origin rpy="0 0 0" xyz="0 0 0" />
+    </collision>
   </link>
   <joint name="laser_joint" type="fixed">
     <parent link="base_link" />
     <child link="laser_link" />
-    <origin xyz="0.0 0.0 0.37733" rpy="0 0 ${radians(-90)}"/>
-  </joint>
-  <link name="laser_link" />
+    <origin xyz="0.0 0.0 0.37733" rpy="0 0 ${radians(-90)}" />
+  </joint>
+  <link name="laser_link">
+    <visual>
+      <origin xyz="0 0 0" rpy="0 0 0" />
+      <geometry>
+        <box size="0.02 0.02 0.001" />
+      </geometry>
+      <material name="dark" />
+    </visual>
+    <collision>
+      <origin xyz="0 0 0" rpy="0 0 0" />
+      <geometry>
+        <box size="0.02 0.02 0.001" />
+      </geometry>
+      <material name="dark" />
+    </collision>
+  </link>
   <joint name="wheel_left_joint" type="continuous">
-    <parent link="base_link"/>
-    <child link="wheel_left_link"/>
-    <origin xyz="0.0 0.08316 0.01004" rpy="-1.57 0 0"/>
-    <axis xyz="0 0 1"/>
+    <parent link="base_link" />
+    <child link="wheel_left_link" />
+    <origin xyz="0.0 0.08316 0.01004" rpy="-1.57 0 0" />
+    <axis xyz="0 0 1" />
   </joint>
   <link name="wheel_left_link">
     <visual>
-      <origin xyz="0 0 0" rpy="1.57 0 0"/>
-      <geometry>
-        <!-- <cylinder length="0.020" radius="0.0254"/> -->
-        <mesh filename="package://jrb_description/meshes/roue.STL" />
-      </geometry>
-      <material name="dark"/>
-    </visual>
+      <origin xyz="0 0 0" rpy="1.57 0 0" />
+      <geometry>
+        <mesh filename="package://jrb_description/urdf/meshes/roue.STL" />
+      </geometry>
+      <material name="dark" />
+    </visual>
+    <collision>
+      <origin xyz="0 0 0" rpy="0 0 0" />
+      <geometry>
+        <cylinder length="0.020" radius="0.0254" />
+      </geometry>
+      <material name="dark" />
+    </collision>
   </link>
   <joint name="wheel_right_joint" type="continuous">
-    <parent link="base_link"/>
-    <child link="wheel_right_link"/>
-    <origin xyz="0.0 -0.08316  0.01004" rpy="-1.57 0 0"/>
-    <axis xyz="0 0 1"/>
+    <parent link="base_link" />
+    <child link="wheel_right_link" />
+    <origin xyz="0.0 -0.08316  0.01004" rpy="-1.57 0 0" />
+    <axis xyz="0 0 1" />
   </joint>
   <link name="wheel_right_link">
-    <visual>
-      <origin xyz="0 0 0" rpy="1.57 0 0"/>
-      <geometry>
-        <!-- <cylinder length="0.018" radius="0.0254"/> -->
-        <mesh filename="package://jrb_description/meshes/roue.STL" />
-      </geometry>
-      <material name="dark"/>
-    </visual>
-    <inertial>
-      <origin xyz="0 0 0" />
-      <mass value="2.8498940e-02" />
-      <inertia ixx="1.1175580e-05" ixy="-4.2369783e-11" ixz="-5.9381719e-09" iyy="1.1192413e-05" iyz="-1.4400107e-11" izz="2.0712558e-05" />
-    </inertial>
+    <collision>
+      <origin xyz="0 0 0" rpy="0 0 0" />
+      <geometry>
+        <cylinder length="0.018" radius="0.0254" />
+      </geometry>
+      <material name="dark" />
+    </collision>
+    <visual>
+      <origin xyz="0 0 0" rpy="1.57 0 0" />
+      <geometry>
+        <mesh filename="package://jrb_description/urdf/meshes/roue.STL" />
+      </geometry>
+      <material name="dark" />
+    </visual>
   </link>
   <joint name="left_tag_joint" type="fixed">
-    <parent link="base_link"/>
-    <child link="left_tag_link"/>
-    <origin xyz="0.091 0.0925 0.0" rpy="0 0 0"/>
+    <parent link="base_link" />
+    <child link="left_tag_link" />
+    <origin xyz="0.091 0.0925 0.0" rpy="0 0 0" />
   </joint>
   <link name="left_tag_link">
     <visual>
-      <origin xyz="0 0 0" rpy="0 0 0"/>
-      <geometry>
-        <box size="0.02 0.02 0.001"/>
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