Commit message: PoC vision OK

File: jrb_description/urdf/robotrouge.urdf.xacro (robot description, xacro)
@@ -38,5 +38,5 @@
     <parent link="base_footprint"/>
     <child link="base_link"/>
-    <origin xyz="0.0 0.0 0.01416" rpy="0 0 0"/>
+    <origin xyz="0.0 0.0 0.0147" rpy="0 0 0"/>
   </joint>
   <link name="base_link">
@@ -60,5 +60,5 @@
     <parent link="base_link"/>
     <child link="wheel_left_link"/>
-    <origin xyz="0.0 0.08316 0" rpy="-1.57 0 0"/>
+    <origin xyz="0.0 0.08316 0.01004" rpy="-1.57 0 0"/>
     <axis xyz="0 0 1"/>
   </joint>
@@ -76,5 +76,5 @@
     <parent link="base_link"/>
     <child link="wheel_right_link"/>
-    <origin xyz="0.0 -0.08316  0.0" rpy="-1.57 0 0"/>
+    <origin xyz="0.0 -0.08316  0.01004" rpy="-1.57 0 0"/>
     <axis xyz="0 0 1"/>
   </joint>
@@ -125,5 +125,5 @@
     <parent link="base_link"/>
     <child link="th_camera_link"/>
-    <origin xyz="0.01468 0.0 0.317" rpy="0 0 0"/>
+    <origin xyz="0.1468 0.0 0.317" rpy="0 0 0"/>
   </joint>
   <link name="th_camera_link">

Commit message: wip gazebo

File: jrb_description/urdf/robotrouge.urdf.xacro (robot description, xacro)
@@ -2,33 +2,21 @@
 <robot name="robotrouge"
   xmlns:xacro="http://ros.org/wiki/xacro">
+  <gazebo>
+      <plugin name="gazebo_ros_joint_state_publisher"
+          filename="libgazebo_ros_joint_state_publisher.so">
+          <update_rate>20</update_rate>
+          <joint_name>slider_joint</joint_name>
+          <joint_name>arm_joint</joint_name>
+      </plugin>
+  </gazebo>
+  <gazebo>
+    <plugin name="gazebo_ros_joint_pose_trajectory"
+        filename="libgazebo_ros_joint_pose_trajectory.so">
+        <update_rate>20</update_rate>
+    </plugin>
+</gazebo>
   <!-- <xacro:include filename="arm.urdf.xacro" /> -->
   <xacro:include filename="colors.xacro" />
   <xacro:include filename="inertial.xacro" />
-  <!-- Webots -->
-  <webots>
-    <device reference="laser_link" type="Lidar">
-      <ros>
-        <enabled>true</enabled>
-        <updateRate>5</updateRate>
-        <topicName>/scan</topicName>
-        <alwaysOn>true</alwaysOn>
-        <frameName>laser_link</frameName>
-      </ros>
-    </device>
-    <plugin type="webots_ros2_control::Ros2Control" />
-  </webots>
-  <ros2_control name="WebotsControl" type="system">
-    <hardware>
-      <plugin>webots_ros2_control::Ros2ControlSystem</plugin>
-    </hardware>
-    <joint name="right_wheel_joint">
-      <state_interface name="position" />
-      <command_interface name="velocity" />
-    </joint>
-    <joint name="left_wheel_joint">
-      <state_interface name="position" />
-      <command_interface name="velocity" />
-    </joint>
-  </ros2_control>
   <!-- BASE LINK -->
   <link name="chassis">

Commit message: fix: use sim time for joint state publisher

File: jrb_description/urdf/robotrouge.urdf.xacro (robot description, xacro)
@@ -2,22 +2,16 @@
 <robot name="robotrouge"
   xmlns:xacro="http://ros.org/wiki/xacro">
-  <gazebo>
-      <plugin name="gazebo_ros_joint_state_publisher"
-          filename="libgazebo_ros_joint_state_publisher.so">
-          <update_rate>20</update_rate>
-          <joint_name>slider_joint</joint_name>
-          <joint_name>arm_joint</joint_name>
-      </plugin>
-  </gazebo>
-  <gazebo>
-    <plugin name="gazebo_ros_joint_pose_trajectory"
-        filename="libgazebo_ros_joint_pose_trajectory.so">
-        <update_rate>20</update_rate>
-    </plugin>
-</gazebo>
   <!-- <xacro:include filename="arm.urdf.xacro" /> -->
   <xacro:include filename="colors.xacro" />
   <xacro:include filename="inertial.xacro" />
   <!-- BASE LINK -->
+  <link name="base_link">
+  </link>
+  <!-- CHASSIS LINK -->
+  <joint name="chassis_joint" type="fixed">
+    <parent link="base_link"/>
+    <child link="chassis"/>
+    <origin xyz="-0.1 0 0"/>
+  </joint>
   <link name="chassis">
     <visual>
@@ -150,4 +144,24 @@
     </collision>
   </link>
+  <gazebo reference="chassis">
+    <material>Gazebo/Orange</material>
+  </gazebo>
+  <gazebo reference="left_wheel">
+    <material>Gazebo/Blue</material>
+  </gazebo>
+  <gazebo reference="right_wheel">
+    <material>Gazebo/Blue</material>
+  </gazebo>
+  <gazebo reference="back_caster_wheel">
+    <material>Gazebo/Black</material>
+    <mu1 value="0.001"/>
+    <mu2 value="0.001"/>
+  </gazebo>
+  <gazebo reference="front_caster_wheel">
+    <material>Gazebo/Black</material>
+    <mu1 value="0.001"/>
+    <mu2 value="0.001"/>
+  </gazebo>
+  <xacro:include filename="gazebo_control.xacro" />
   <!-- <link name="base_footprint">
     <visual>
