Commit message: wip: urdf

File: jrb_description/urdf/colors.xacro (robot description, xacro)
@@ -31,3 +31,6 @@
         <color rgba="1.0 1.0 1.0 1.0" />
     </material>
+    <material name="yellow">
+        <color rgba="1.0 1.0 0.0 1.0" />
+    </material>
 </robot>

File: jrb_description/urdf/gazebo.xacro (robot description, xacro)
@@ -1,84 +1,25 @@
 <?xml version="1.0"?>
 <robot xmlns:xacro="http://www.ros.org/wiki/xacro">
-    <!-- This file demonstrates the use of some <gazebo> tags -->
-    <!-- To include it add the following line -->
-    <!-- <xacro:include filename="example_gazebo.xacro" /> -->
-    <!-- Gazebo is unable to use the same <material> tags that are already in the URDF (that RViz uses). -->
-    <!-- Instead, we need to add gazebo tags for our links that refer to Gazebo materials -->
-    <gazebo reference="base_link">
-        <material>Gazebo/Green</material>
+    <gazebo reference="chassis">
+        <material>Gazebo/Orange</material>
     </gazebo>
-    <gazebo reference="slider_link">
+    <gazebo reference="carter">
+        <material>Gazebo/Yellow</material>
+    </gazebo>
+    <gazebo reference="left_wheel">
         <material>Gazebo/Blue</material>
     </gazebo>
-    <gazebo reference="arm_link">
-        <material>Gazebo/Orange</material>
+    <gazebo reference="right_wheel">
+        <material>Gazebo/Blue</material>
     </gazebo>
-    <!-- Gazebo requires the use of plugins to interact with other systems such as ROS. -->
-    <!-- This plugin will publish the joint_states for the selected joints
-            (which robot_state_publisher can then use to broadcast the approprate tf). -->
-    <gazebo>
-        <plugin name="gazebo_ros_joint_state_publisher"
-            filename="libgazebo_ros_joint_state_publisher.so">
-            <update_rate>20</update_rate>
-            <joint_name>slider_joint</joint_name>
-            <joint_name>arm_joint</joint_name>
-        </plugin>
+    <gazebo reference="front_caster_wheel">
+        <material>Gazebo/White</material>
+        <mu1 value="0.001"/>
+        <mu2 value="0.001"/>
     </gazebo>
-    <!-- This plugin will read a JointTrajectory message from the /set_joint_trajectory topic
-            and move the machine accordingly. It's a bit clunky but it works. -->
-    <!-- You'll probably want to add damping to the joints to stop them it flopping around.
-            e.g. <dynamics damping="10.0" friction="10.0"/> -->
-    <!-- Here's an example message to publish to test it:
-            ros2 topic pub -1 /set_joint_trajectory trajectory_msgs/msg/JointTrajectory  '{header: {frame_id: world}, joint_names: [slider_joint, arm_joint], points: [  {positions: {0.8,0.6}} ]}' -->
-    <gazebo>
-        <plugin name="gazebo_ros_joint_pose_trajectory"
-            filename="libgazebo_ros_joint_pose_trajectory.so">
-            <update_rate>2</update_rate>
-        </plugin>
-    </gazebo>
-    <!-- The next section shows an example of adding a sensor, in this case a depth camera. -->
-    <!-- Due to a quirk of how cameras work, an extra joint/link is required to create an
-            "optical frame" for the sensor. That isn't the focus for this tutorial, but you can
-            look at https://www.ros.org/reps/rep-0103.html#suffix-frames for slightly more information. -->
-    <!-- First, create the link and joint for the optical frame -->
-    <joint name="camera_optical_joint" type="fixed">
-        <origin xyz="0 0 0" rpy="-1.571 0 -1.571" />
-        <parent link="camera_link" />
-        <child link="camera_link_optical" />
-    </joint>
-    <link name="camera_link_optical"></link>
-    <!-- Add a gazebo tag for the ORIGINAL camera_link (but in the plugin we reference the optical frame so that ROS can orient things correctly) -->
-    <!-- Within the gazebo tag we have the sensor tag, and inside that there is (among other things) the camera tag with the camera parameters,
-            and the plugin tag with some extra parameters the plugin needs. -->
-    <!-- Note that although visualise is set to true, it won't actually visualise the depth camera in gazebo. To see the preview,
-            try swapping "depth" to "camera"-->
-    <gazebo reference="camera_link">
-        <sensor type="depth" name="my_camera">
-            <update_rate>20</update_rate>
-            <visualize>true</visualize>
-            <camera name="cam">
-                <horizontal_fov>1.3962634</horizontal_fov>
-                <image>
-                    <width>640</width>
-                    <height>480</height>
-                    <format>R8B8G8</format>
-                </image>
-                <clip>
-                    <near>0.02</near>
-                    <far>300</far>
-                </clip>
-                <noise>
-                    <type>gaussian</type>
-                    <mean>0.0</mean>
-                    <stddev>0.007</stddev>
-                </noise>
-            </camera>
-            <plugin name="camera_controller" filename="libgazebo_ros_camera.so">
-                <frame_name>camera_link_optical</frame_name>
-                <min_depth>0.1</min_depth>
-                <max_depth>500</max_depth>
-            </plugin>
-        </sensor>
+    <gazebo reference="back_caster_wheel">
+        <material>Gazebo/White</material>
+        <mu1 value="0.001"/>
+        <mu2 value="0.001"/>
     </gazebo>
 </robot>

File: jrb_description/urdf/robotrouge.urdf.xacro (robot description, xacro)
@@ -2,372 +2,241 @@
 <robot name="robotrouge"
   xmlns:xacro="http://ros.org/wiki/xacro">
-  <!-- <xacro:include filename="arm.urdf.xacro" /> -->
-  <xacro:include filename="colors.xacro" />
-  <xacro:include filename="inertial.xacro" />
-  <!-- BASE LINK -->
-  <link name="base_link">
-  </link>
-  <!-- CHASSIS LINK -->
-  <joint name="chassis_joint" type="fixed">
-    <parent link="base_link"/>
-    <child link="chassis"/>
-    <origin xyz="-0.1 0 0"/>
-  </joint>
-  <link name="chassis">
-    <visual>
-      <origin xyz="0 0 0.075" />
-      <geometry>
-        <box size="0.3 0.3 0.15" />
-      </geometry>
-      <material name="white" />
-    </visual>
-    <collision>
-      <origin xyz="0 0 0.075" />
-      <geometry>
-        <box size="0.3 0.3 0.15" />
-      </geometry>
-    </collision>
-    <xacro:inertial_box mass="0.5" x="0.3" y="0.3" z="0.15">
-      <origin xyz="0 0 0.075" rpy="0 0 0" />
-    </xacro:inertial_box>
-  </link>
-  <!-- LEFT WHEEL LINK -->
-  <joint name="left_wheel_joint" type="continuous">
-    <parent link="chassis" />
-    <child link="left_wheel" />
-    <origin xyz="0 0.15 0" rpy="-${pi/2} 0 0" />
-    <axis xyz="0 0 1" />
-  </joint>
-  <link name="left_wheel">
-    <visual>
-      <geometry>
-        <cylinder radius="0.0254" length="0.02" />
-      </geometry>
-      <material name="blue" />
-    </visual>
-    <collision>
-      <geometry>
-        <cylinder radius="0.0254" length="0.02" />
-      </geometry>
-    </collision>
-    <xacro:inertial_cylinder mass="0.1" length="0.02" radius="0.0254">
-      <origin xyz="0 0 0" rpy="0 0 0" />
-    </xacro:inertial_cylinder>
-  </link>
-  <!-- RIGHT WHEEL LINK -->
-  <joint name="right_wheel_joint" type="continuous">
-    <parent link="chassis" />
-    <child link="right_wheel" />
-    <origin xyz="0 -0.15 0" rpy="${pi/2} 0 0" />
-    <axis xyz="0 0 -1" />
-  </joint>
-  <link name="right_wheel">
-    <visual>
-      <geometry>
-        <cylinder radius="0.0254" length="0.02" />
-      </geometry>
-      <material name="blue" />
-    </visual>
-    <collision>
-      <geometry>
-        <cylinder radius="0.0254" length="0.02" />
-      </geometry>
-    </collision>
-    <xacro:inertial_cylinder mass="0.1" length="0.02" radius="0.0254">
-      <origin xyz="0 0 0" rpy="0 0 0" />
-    </xacro:inertial_cylinder>
-  </link>
-  <!-- FRONT CASTER WHEEL LINK -->
-  <joint name="front_caster_wheel_joint" type="fixed">
-    <parent link="chassis" />
-    <child link="front_caster_wheel" />
-    <origin xyz="0.12 0 0" />
-  </joint>
-  <link name="front_caster_wheel">
-    <visual>
-      <geometry>
-        <sphere radius="0.0254" />
-      </geometry>
-      <material name="black" />
-    </visual>
-    <collision>
-      <geometry>
-        <sphere radius="0.0254" />
-      </geometry>
-    </collision>
-    <xacro:inertial_sphere mass="0.1" radius="0.0254">
-      <origin xyz="0 0 0" rpy="0 0 0" />
-    </xacro:inertial_sphere>
-  </link>
-  <!-- BACK CASTER WHEEL LINK -->
-  <joint name="back_caster_wheel_joint" type="fixed">
-    <parent link="chassis" />
-    <child link="back_caster_wheel" />
-    <origin xyz="-0.12 0 0" />
-  </joint>
-  <link name="back_caster_wheel">
-    <visual>
-      <geometry>
-        <sphere radius="0.0254" />
-      </geometry>
-      <material name="black" />
-    </visual>
-    <collision>
-      <geometry>
-        <sphere radius="0.0254" />
-      </geometry>
-    </collision>
-    <xacro:inertial_sphere mass="0.1" radius="0.0254">
-      <origin xyz="0 0 0" rpy="0 0 0" />
-    </xacro:inertial_sphere>
-  </link>
-  <!-- LASER LINK  -->
-  <joint name="laser_joint" type="fixed">
-    <parent link="chassis" />
-    <child link="laser_link" />
-    <origin xyz="0.0 0.0 0.37733" rpy="0 0 ${-pi/2}" />
-  </joint>
-  <link name="laser_link">
-    <visual>
-      <origin xyz="0 0 0" rpy="0 0 0" />
-      <geometry>
-        <box size="0.02 0.02 0.001" />
-      </geometry>
-      <material name="dark" />
-    </visual>
-    <collision>
-      <origin xyz="0 0 0" rpy="0 0 0" />
-      <geometry>
-        <box size="0.02 0.02 0.001" />
-      </geometry>
-      <material name="dark" />
-    </collision>
-  </link>
-  <gazebo reference="chassis">
-    <material>Gazebo/Orange</material>
-  </gazebo>
-  <gazebo reference="left_wheel">
-    <material>Gazebo/Blue</material>
-  </gazebo>
-  <gazebo reference="right_wheel">
-    <material>Gazebo/Blue</material>
-  </gazebo>
-  <gazebo reference="back_caster_wheel">
-    <material>Gazebo/Black</material>
-    <mu1 value="0.001"/>
-    <mu2 value="0.001"/>
-  </gazebo>
-  <gazebo reference="front_caster_wheel">
-    <material>Gazebo/Black</material>
-    <mu1 value="0.001"/>
-    <mu2 value="0.001"/>
-  </gazebo>
-  <xacro:include filename="gazebo_control.xacro" />
-  <!-- <link name="base_footprint">
-    <visual>
-      <origin xyz="0 0 0.02" rpy="0 0 0" />
-      <geometry>
-        <mesh filename="package://jrb_description/urdf/meshes/carter.STL" />
-      </geometry>
-    </visual>
-    <collision>
-      <origin xyz="0 0 0.22" rpy="0 0 0" />
-      <geometry>
-        <box size="0.2 0.27 0.4" />
-      </geometry>
-      <material name="light_black" />
-    </collision>
-  </link>
-  <joint name="base_joint" type="fixed">
-    <parent link="base_footprint" />
-    <child link="base_link" />
-    <origin xyz="0.0 0.0 0.0147" rpy="0 0 0" />
-  </joint>
-  <link name="base_link">
-    <visual>
-      <origin xyz="0 0 -0.003" rpy="0 0 3.14" />
-      <geometry>
-        <mesh filename="package://jrb_description/urdf/meshes/base.STL" />
-      </geometry>
-      <material name="light_black" />
-    </visual>
-    <collision>
-      <origin xyz="0 0 0" rpy="0 0 0" />
-      <geometry>
-        <box size="0.2 0.27 0.01" />
-      </geometry>
-      <material name="light_black" />
-    </collision>
-  </link>
-  <joint name="caster_front_joint" type="fixed">
-    <parent link="base_footprint" />
-    <child link="caster_front_link" />
-    <origin rpy="0 0 0" xyz="0.09 0.0 0.01" />
-  </joint>
-  <link name="caster_front_link">
-    <visual>
-      <origin rpy="0 0 0" xyz="0 0 0" />
-      <geometry>
-        <sphere radius="0.01" />
-      </geometry>
-      <material name="Black" />
-    </visual>
-    <collision>
-      <geometry>
-        <sphere radius="0.01" />
-      </geometry>
-      <origin rpy="0 0 0" xyz="0 0 0" />
-    </collision>
-  </link>
-  <joint name="caster_back_joint" type="fixed">
-    <parent link="base_footprint" />
-    <child link="caster_back_link" />
-    <origin rpy="0 0 0" xyz="-0.09 0.0 0.01" />
-  </joint>
-  <link name="caster_back_link">
-    <visual>
-      <origin rpy="0 0 0" xyz="0 0 0" />
-      <geometry>
-        <sphere radius="0.01" />
-      </geometry>
-      <material name="Black" />
-    </visual>
-    <collision>
-      <geometry>
-        <sphere radius="0.01" />
-      </geometry>
-      <origin rpy="0 0 0" xyz="0 0 0" />
-    </collision>
-  </link>
-  <joint name="laser_joint" type="fixed">
-    <parent link="base_link" />
-    <child link="laser_link" />
-    <origin xyz="0.0 0.0 0.37733" rpy="0 0 ${radians(-90)}" />
-  </joint>
-  <link name="laser_link">
-    <visual>
-      <origin xyz="0 0 0" rpy="0 0 0" />
-      <geometry>
-        <box size="0.02 0.02 0.001" />
-      </geometry>
-      <material name="dark" />
-    </visual>
-    <collision>
-      <origin xyz="0 0 0" rpy="0 0 0" />
-      <geometry>
-        <box size="0.02 0.02 0.001" />
-      </geometry>
-      <material name="dark" />
-    </collision>
-  </link>
-  <joint name="wheel_left_joint" type="continuous">
-    <parent link="base_link" />
-    <child link="wheel_left_link" />
-    <origin xyz="0.0 0.08316 0.01004" rpy="-1.57 0 0" />
-    <axis xyz="0 0 1" />
-  </joint>
-  <link name="wheel_left_link">
-    <visual>
-      <origin xyz="0 0 0" rpy="1.57 0 0" />
-      <geometry>
-        <mesh filename="package://jrb_description/urdf/meshes/roue.STL" />
-      </geometry>
-      <material name="dark" />
-    </visual>
-    <collision>
-      <origin xyz="0 0 0" rpy="0 0 0" />
-      <geometry>
-        <cylinder length="0.020" radius="0.0254" />
-      </geometry>
-      <material name="dark" />
-    </collision>
-  </link>
-  <joint name="wheel_right_joint" type="continuous">
-    <parent link="base_link" />
-    <child link="wheel_right_link" />
-    <origin xyz="0.0 -0.08316  0.01004" rpy="-1.57 0 0" />
-    <axis xyz="0 0 1" />
-  </joint>
-  <link name="wheel_right_link">
-    <collision>
-      <origin xyz="0 0 0" rpy="0 0 0" />
-      <geometry>
-        <cylinder length="0.018" radius="0.0254" />
-      </geometry>
-      <material name="dark" />
-    </collision>
-    <visual>
-      <origin xyz="0 0 0" rpy="1.57 0 0" />
-      <geometry>
-        <mesh filename="package://jrb_description/urdf/meshes/roue.STL" />
-      </geometry>
-      <material name="dark" />
-    </visual>
-  </link>
-  <joint name="left_tag_joint" type="fixed">
-    <parent link="base_link" />
-    <child link="left_tag_link" />
-    <origin xyz="0.091 0.0925 0.0" rpy="0 0 0" />
-  </joint>
-  <link name="left_tag_link">
-    <visual>
-      <origin xyz="0 0 0" rpy="0 0 0" />
-      <geometry>
-        <box size="0.02 0.02 0.001" />
-      </geometry>
-      <material name="dark" />
-    </visual>
-    <collision>
-      <origin xyz="0 0 0" rpy="0 0 0" />
-      <geometry>
-        <box size="0.02 0.02 0.001" />
-      </geometry>
-      <material name="dark" />
-    </collision>
-  </link>
-  <joint name="right_tag_joint" type="fixed">
-    <parent link="base_link" />
-    <child link="right_tag_link" />
-    <origin xyz="0.091 -0.0925 0.0" rpy="0 0 0" />
-  </joint>
-  <link name="right_tag_link">
-    <visual>
-      <origin xyz="0 0 0" rpy="0 0 0" />
-      <geometry>
-        <box size="0.02 0.02 0.001" />
-      </geometry>
-      <material name="dark" />
-    </visual>
-    <collision>
-      <origin xyz="0 0 0" rpy="0 0 0" />
-      <geometry>
-        <box size="0.02 0.02 0.001" />
-      </geometry>
-      <material name="dark" />
-    </collision>
-  </link>
-  <joint name="th_camera_joint" type="fixed">
-    <parent link="base_link" />
-    <child link="th_camera_link" />
-    <origin xyz="0.1468 0.0 0.317" rpy="0 0 0" />
-  </joint>
-  <link name="th_camera_link">
-    <visual>
-      <origin xyz="0 0 0" rpy="0 0 0" />
-      <geometry>
-        <box size="0.02 0.02 0.001" />
-      </geometry>
-      <material name="dark" />
-    </visual>
-    <collision>
-      <origin xyz="0 0 0" rpy="0 0 0" />
-      <geometry>
-        <box size="0.02 0.02 0.001" />
-      </geometry>
-      <material name="dark" />
-    </collision>
-  </link> -->
-  <!-- Arms -->
-  <!-- <xacro:arm name="left" xyz="0.054 0.11275 0.029375" origin="0.0865 0.11275 0" />
-  <xacro:arm name="right" xyz="0.054 -0.11275 0.029375" origin="0.0865 -0.11275 0" /> -->
+    <!-- <xacro:include filename="arm.urdf.xacro" /> -->
+    <xacro:include filename="colors.xacro" />
+    <xacro:include filename="inertial.xacro" />
+    <xacro:arg name="display_meshes" default="True"/>
+    <xacro:property name="chassis_length" value="0.2"/>
+    <xacro:property name="chassis_width" value="0.275"/>
+    <xacro:property name="chassis_height" value="0.006"/>
+    <xacro:property name="chassis_mass" value="1.0"/>
+    <xacro:property name="carter_length" value="0.17"/>
+    <xacro:property name="carter_width" value="0.275"/>
+    <xacro:property name="carter_height" value="0.33"/>
+    <xacro:property name="carter_mass" value="0.1"/>
+    <xacro:property name="carter_offset_x" value="0.045"/>
+    <xacro:property name="wheel_radius" value="0.0254"/>
+    <xacro:property name="wheel_thickness" value="0.018"/>
+    <xacro:property name="wheel_mass" value="0.05"/>
+    <xacro:property name="wheel_offset_x" value="0.0"/>
+    <xacro:property name="wheel_offset_y" value="0.08316"/>
+    <xacro:property name="wheel_offset_z" value="0.0"/>
+    <xacro:property name="caster_wheel_radius" value="0.008"/>
+    <xacro:property name="caster_wheel_mass" value="0.01"/>
+    <xacro:property name="caster_wheel_offset_x" value="0.085"/>
+    <xacro:property name="caster_wheel_offset_z" value="${wheel_offset_z - wheel_radius + caster_wheel_radius}"/>
+    <!-- BASE LINK -->
+    <link name="base_link">
+    </link>
+    <!-- BASE_FOOTPRINT LINK -->
+    <joint name="base_footprint_joint" type="fixed">
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