Commit message: feat: add lidar

File: jrb_description/urdf/gazebo.xacro (robot description, xacro)
@@ -23,3 +23,31 @@
         <mu2 value="0.001"/>
     </gazebo>
+    <gazebo reference="laser_link">
+        <material>Gazebo/Red</material>
+        <sensor name="laser_link" type="ray">
+            <pose> 0 0 0 0 0 0 </pose>
+            <visualize>false</visualize>
+            <update_rate>10</update_rate>
+            <ray>
+                <scan>
+                    <horizontal>
+                        <samples>360</samples>
+                        <min_angle>-3.14</min_angle>
+                        <max_angle>3.14</max_angle>
+                    </horizontal>
+                </scan>
+                <range>
+                    <min>0.3</min>
+                    <max>12</max>
+                </range>
+            </ray>
+            <plugin name="laser_controller" filename="libgazebo_ros_ray_sensor.so">
+                <ros>
+                    <argument>~/out:=scan</argument>
+                </ros>
+                <output_type>sensor_msgs/LaserScan</output_type>
+                <frame_name>laser_link</frame_name>
+            </plugin>
+        </sensor>
+    </gazebo>
 </robot>

File: jrb_description/urdf/robotrouge.urdf.xacro (robot description, xacro)
@@ -25,4 +25,5 @@
     <xacro:property name="caster_wheel_offset_x" value="0.085"/>
     <xacro:property name="caster_wheel_offset_z" value="${wheel_offset_z - wheel_radius + caster_wheel_radius}"/>
+    <xacro:property name="lidar_height" value="0.37733"/>
     <!-- BASE LINK -->
     <link name="base_link">
@@ -55,5 +56,4 @@
                     <box size="${chassis_length} ${chassis_width} ${chassis_height}"/>
                 </geometry>
-                <material name="orange"/>
             </xacro:unless>
             <material name="orange"/>
@@ -238,4 +238,5 @@
         </visual>
     </link>
+    <xacro:include filename="lidar.xacro" />
     <xacro:include filename="gazebo.xacro" />
     <xacro:include filename="gazebo_control.xacro" />

Commit message: wip: add eurobot table in gazebo; clean sample_detector; add twist_mux

File: jrb_description/urdf/gazebo.xacro (robot description, xacro)
@@ -1,4 +1,5 @@
 <?xml version="1.0"?>
 <robot xmlns:xacro="http://www.ros.org/wiki/xacro">
+    <!-- CORE -->
     <gazebo reference="chassis">
         <material>Gazebo/Orange</material>
@@ -23,4 +24,5 @@
         <mu2 value="0.001"/>
     </gazebo>
+    <!-- LIDAR -->
     <gazebo reference="laser_link">
         <material>Gazebo/Red</material>
@@ -51,3 +53,27 @@
         </sensor>
     </gazebo>
+    <!-- CAMERA -->
+    <gazebo reference="camera_link">
+        <material>Gazebo/Black</material>
+        <sensor name="camera" type="camera">
+            <pose> 0 0 0 0 0 0 </pose>
+            <visualize>false</visualize>
+            <update_rate>5</update_rate>
+            <camera>
+                <horizontal_fov>1.089</horizontal_fov>
+                <image>
+                    <format>R8G8B8</format>
+                    <width>640</width>
+                    <height>480</height>
+                </image>
+                <clip>
+                    <near>0.05</near>
+                    <far>8.0</far>
+                </clip>
+            </camera>
+            <plugin name="camera_controller" filename="libgazebo_ros_camera.so">
+                <frame_name>camera_link_optical</frame_name>
+            </plugin>
+        </sensor>
+    </gazebo>
 </robot>

File: jrb_description/urdf/gazebo_control.xacro (robot description, xacro)
@@ -15,5 +15,5 @@
             <robot_base_frame>base_link</robot_base_frame>
             <publish_odom>true</publish_odom>
-            <publish_odom_tf>true</publish_odom_tf>
+            <publish_odom_tf>false</publish_odom_tf>
             <publish_wheel_tf>true</publish_wheel_tf>
         </plugin>

File: jrb_description/urdf/robotrouge.urdf.xacro (robot description, xacro)
@@ -216,9 +216,8 @@
     <link name="left_tag_link">
         <visual>
-            <origin xyz="0 0 0.0005" rpy="0 0 0"/>
-            <geometry>
-                <box size="0.02 0.02 0.001"/>
-            </geometry>
-            <material name="dark"/>
+            <origin xyz="0 0 0" rpy="0 0 0"/>
+                <geometry>
+                    <mesh filename="package://jrb_description/urdf/meshes/tag/tag_left.dae" />
+                </geometry>
         </visual>
     </link>
@@ -231,12 +230,12 @@
     <link name="right_tag_link">
         <visual>
-            <origin xyz="0 0 0.0005" rpy="0 0 0"/>
-            <geometry>
-                <box size="0.02 0.02 0.001"/>
-            </geometry>
-            <material name="dark"/>
+            <origin xyz="0 0 0" rpy="0 0 0"/>
+                <geometry>
+                    <mesh filename="package://jrb_description/urdf/meshes/tag/tag_right.dae" />
+                </geometry>
         </visual>
     </link>
     <xacro:include filename="lidar.xacro" />
+    <xacro:include filename="camera.xacro" />
     <xacro:include filename="gazebo.xacro" />
     <xacro:include filename="gazebo_control.xacro" />
